Commit message: p2: update

File: p2/old_robot_models/robot_v1/urdf/robot_v1.urdf (robot description, URDF)
Before this commit: robot robot_v1, 5 links, 4 joints
Links:
- link cuerpo_link: geometry collision mesh filename=../meshes/stl/Cubo.009.stl scale=0.90000 0.70000 0.50000; visual mesh filename=../meshes/stl/Cubo.009.stl scale=0.90000 0.70000 0.50000
- link rueda_a_d_link: geometry collision mesh filename=../meshes/stl/Cilindro.stl scale=0.55000 0.55000 0.15000; visual mesh filename=../meshes/stl/Cilindro.stl scale=0.55000 0.55000 0.15000
- link rueda_a_i_link: geometry collision mesh filename=../meshes/stl/Cilindro.stl scale=0.55000 0.55000 0.15000; visual mesh filename=../meshes/stl/Cilindro.stl scale=0.55000 0.55000 0.15000
- link rueda_d_l_link: geometry collision mesh filename=../meshes/stl/Cilindro.stl scale=0.55000 0.55000 0.15000; visual mesh filename=../meshes/stl/Cilindro.stl scale=0.55000 0.55000 0.15000
- link rueda_d_r_link: geometry collision mesh filename=../meshes/stl/Cilindro.stl scale=0.55000 0.55000 0.15000; visual mesh filename=../meshes/stl/Cilindro.stl scale=0.55000 0.55000 0.15000
Joints:
- joint rueda_a_d_link_joint: origin xyz=-1.00000 2.74000 -1.65000 rpy=0.00000 -1.57080 0.00000 -> xyz=-1.00000 2.74000 -1.65000 rpy=-0.00000 1.57080 0.00000
- joint rueda_d_r_link_joint: origin xyz=-1.00000 -0.26000 -1.65000 rpy=0.00000 -1.57080 0.00000 -> xyz=-1.00000 -0.26000 -1.65000 rpy=-0.00000 1.57080 0.00000
